Commit message: updated urdf

File: ballie_bot_description/urdf/ballie_bot.urdf.xacro (robot description, xacro)
@@ -29,26 +29,39 @@
     <origin xyz="0.0 0.0 ${-(wheel_radius+wheel_zoff)}" rpy="0 0 0"/>
   </joint>
-    <!-- Wheels -->
-  <xacro:macro name="wheel" params="prefix x_reflect y_reflect">
-    <link name="${prefix}_link">
-      <visual>
-        <origin xyz="0 0 0" rpy="${pi/2} 0 0"/>
-        <geometry>
-            <cylinder radius="${wheel_radius}" length="${wheel_width}"/>
-        </geometry>
-        <material name="Gray">
-          <color rgba="0.5 0.5 0.5 1.0"/>
-        </material>
-      </visual>
-    </link>
-    <joint name="${prefix}_joint" type="continuous">
-      <parent link="base_link"/>
-      <child link="${prefix}_link"/>
-      <origin xyz="${x_reflect*wheel_xoff} ${y_reflect*(base_width/2+wheel_ygap)} ${-wheel_zoff}" rpy="0 0 0"/>
-      <axis xyz="0 1 0"/>
-    </joint>
-  </xacro:macro>
-  <xacro:wheel prefix="drivewhl_l" x_reflect="-1" y_reflect="1" />
-  <xacro:wheel prefix="drivewhl_r" x_reflect="-1" y_reflect="-1" />
+  <!-- wheels -->
+  <link name="drivewhl_l_link">
+    <visual>
+      <origin xyz="0 0 0" rpy="${pi/2} 0 0"/>
+      <geometry>
+          <cylinder radius="${wheel_radius}" length="${wheel_width}"/>
+      </geometry>
+      <material name="Gray">
+        <color rgba="0.5 0.5 0.5 1.0"/>
+      </material>
+    </visual>
+  </link>
+  <joint name="$drivewhl_l_joint" type="continuous">
+    <parent link="base_link"/>
+    <child link="drivewhl_l_link"/>
+    <origin xyz="${1*wheel_xoff} ${1*(base_width/2+wheel_ygap)} ${-wheel_zoff}" rpy="0 0 0"/>
+    <axis xyz="0 1 0"/>
+  </joint>
+  <link name="drivewhl_r_link">
+    <visual>
+      <origin xyz="0 0 0" rpy="${pi/2} 0 0"/>
+      <geometry>
+        <cylinder radius="${wheel_radius}" length="${wheel_width}"/>
+      </geometry>
+      <material name="Gray">
+        <color rgba="0.5 0.5 0.5 1.0"/>
+      </material>
+    </visual>
+  </link>
+  <joint name="$drivewhl_r_joint" type="continuous">
+    <parent link="base_link"/>
+    <child link="drivewhl_r_link"/>
+    <origin xyz="${-1*wheel_xoff} ${1*(base_width/2+wheel_ygap)} ${-wheel_zoff}" rpy="0 0 0"/>
+    <axis xyz="0 1 0"/>
+  </joint>
     <!-- Caster Wheel -->
   <link name="front_caster">
